Commit message: add current arm configuration

File: svenzva_description/robots/svenzva_arm.urdf (robot description, URDF)
Before this commit: robot revel, 11 links, 10 joints
Links:
- removed link ee_link
- removed link finger_joint_2
- removed link finger_link_1
- removed link link_6
Joints:
- removed joint ee_joint
- removed joint finger_joint_1
- removed joint finger_joint_2
- removed joint joint_6

Commit message: ik fast arm sovler changes

File: svenzva_description/robots/svenzva_arm.urdf (robot description, URDF)
Before this commit: robot revel, 7 links, 6 joints
Links:
- added link camera_link
Joints:
- added joint camera_joint: type fixed, parent link_5, child camera_link, origin xyz=0.06 -0.004452 0.06 rpy=0 0 0
